Commit message: Added  simple urdf and modified my_robot urdf (Error of urdf not spawning in gazebo remaining)

File: src/robot_simulation/urdf/my_robot.urdf (robot description, URDF)
Before this commit: robot my_robot, 12 links, 11 joints
Links:
- removed link left_bogie
- removed link left_rocker
- removed link right_bogie
- removed link right_rocker
- link base_link: mass None -> 20.0
- link comp_1: mass None -> 10.0
- link laser_link: mass None -> 1.0
- link left_front_wheel: mass None -> 2.0
- link left_rear_wheel: mass None -> 2.0
- link right_front_wheel: mass None -> 2.0
- link right_rear_wheel: mass None -> 2.0
Joints:
- removed joint left_bogie_joint
- removed joint left_rocker_joint
- removed joint right_bogie_joint
- removed joint right_rocker_joint
