Commit message: Added URDF for Back rocker

File: src/robot_simulation/urdf/rover.urdf (robot description, URDF)
Before this commit: robot my_robot, 3 links, 2 joints
Links:
- added link back_rocker_left_link; visual box size=0.03 0.03 0.2
- added link back_rocker_link; visual box size=0.03 0.632 0.03
- added link back_rocker_right_link; visual box size=0.03 0.03 0.2
Joints:
- added joint back_rocker_back_rocker_left_joint: type fixed, parent back_rocker_link, child back_rocker_left_link, origin xyz=-0.03 0.301 -0.085 rpy=0.0 0.0 0.0
- added joint back_rocker_back_rocker_right_joint: type fixed, parent back_rocker_link, child back_rocker_right_link, origin xyz=-0.03 -0.301 -0.085 rpy=0.0 0.0 0.0
- added joint base_back_rocker_joint: type revolute, parent base_link, child back_rocker_link, origin xyz=-0.425 0.0 0.0 rpy=0.0 0.0 0.0, axis 1.0 0.0 0.0, limit lower=-0.349 upper=0.349 effort=0.0 velocity=0.0

Commit message: Added URDF for Left Front rocker

File: src/robot_simulation/urdf/rover.urdf (robot description, URDF)
Before this commit: robot my_robot, 6 links, 5 joints
Links:
- added link backward_left_front_rocker_link; visual box size=0.3 0.03 0.03
- added link forward_left_front_rocker_link; visual box size=0.33 0.03 0.03
Joints:
- added joint base_forward_left_front_rocker_joint: type revolute, parent base_link, child forward_left_front_rocker_link, origin xyz=0.225 0.267 0.015 rpy=0.0 0.785 0.0, axis 0.0 1.0 0.0, limit lower=-0.523 upper=0.523 effort=0.0 velocity=0.0
- added joint forward_left_front_rocker_backward_left_front_rocker_joint: type fixed, parent forward_left_front_rocker_link, child backward_left_front_rocker_link, origin xyz=0.005 0.0 -0.015 rpy=0.0 -1.57 0.0

Commit message: Added URDF for Right Front rocker

File: src/robot_simulation/urdf/rover.urdf (robot description, URDF)
Before this commit: robot my_robot, 8 links, 7 joints
Links:
- added link backward_right_front_rocker_link; visual box size=0.3 0.03 0.03
- added link forward_right_front_rocker_link; visual box size=0.33 0.03 0.03
Joints:
- added joint base_forward_right_front_rocker_joint: type revolute, parent base_link, child forward_right_front_rocker_link, origin xyz=0.225 -0.282 0.015 rpy=0.0 0.785 0.0, axis 0.0 1.0 0.0, limit lower=-0.523 upper=0.523 effort=0.0 velocity=0.0
- added joint forward_right_front_rocker_backward_right_front_rocker_joint: type fixed, parent forward_right_front_rocker_link, child backward_right_front_rocker_link, origin xyz=0.005 0.0 -0.015 rpy=0.0 -1.57 0.0
- joint base_forward_left_front_rocker_joint: origin xyz=0.225 0.267 0.015 rpy=0.0 0.785 0.0 -> xyz=0.225 0.282 0.015 rpy=0.0 0.785 0.0

Commit message: Added URDF for Front motored wheels

File: src/robot_simulation/urdf/rover.urdf (robot description, URDF)
Before this commit: robot my_robot, 10 links, 9 joints
Links:
- added link left_front_wheel_link; visual cylinder length=0.055 radius=0.127
- added link right_front_wheel_link; visual cylinder length=0.055 radius=0.127
Joints:
- added joint forward_left_front_rocker_left_front_wheel_joint: type continuous, parent forward_left_front_rocker_link, child left_front_wheel_link, origin xyz=0.31 0.0825 0.0 rpy=-1.57 0.0 0.0, axis 0.0 0.0 1.0
- added joint forward_right_front_rocker_right_front_wheel_joint: type continuous, parent forward_right_front_rocker_link, child right_front_wheel_link, origin xyz=0.31 -0.0825 0.0 rpy=1.57 0.0 0.0, axis 0.0 0.0 1.0

Commit message: Added URDF for Back motored wheels

File: src/robot_simulation/urdf/rover.urdf (robot description, URDF)
Before this commit: robot my_robot, 12 links, 11 joints
Links:
- added link left_back_wheel_link; visual cylinder length=0.055 radius=0.127
- added link right_back_wheel_link; visual cylinder length=0.055 radius=0.127
Joints:
- added joint back_rocker_left_left_back_wheel_joint: type continuous, parent back_rocker_left_link, child left_back_wheel_link, origin xyz=0.0 0.0825 -0.09 rpy=1.57 0.0 0.0, axis 0.0 0.0 -1.0
- added joint back_rocker_right_right_back_wheel_joint: type continuous, parent back_rocker_right_link, child right_back_wheel_link, origin xyz=0.0 -0.0825 -0.09 rpy=-1.57 0.0 0.0, axis 0.0 0.0 1.0
- joint forward_right_front_rocker_right_front_wheel_joint: axis 0.0 0.0 1.0 -> 0.0 0.0 -1.0

Commit message: Added URDF for pneumatic motored wheels

File: src/robot_simulation/urdf/rover.urdf (robot description, URDF)
Before this commit: robot my_robot, 14 links, 13 joints
Links:
- added link left_pneumatic_wheel_link; visual cylinder length=0.055 radius=0.127
- added link right_pneumatic_wheel_link; visual cylinder length=0.055 radius=0.127
Joints:
- added joint backward_left_front_rocker_left_pneumatic_wheel_joint: type continuous, parent backward_left_front_rocker_link, child left_pneumatic_wheel_link, origin xyz=-0.29 0.0555 0.0 rpy=-1.57 0.0 0.0, axis 0.0 0.0 1.0
- added joint backward_right_front_rocker_right_pneumatic_wheel_joint: type continuous, parent backward_right_front_rocker_link, child right_pneumatic_wheel_link, origin xyz=-0.29 -0.0555 0.0 rpy=1.57 0.0 0.0, axis 0.0 0.0 -1.0

Commit message: Added collision for converting into SDF

File: src/robot_simulation/urdf/rover.urdf (robot description, URDF)
Before this commit: robot my_robot, 16 links, 15 joints
Links:
- link back_rocker_left_link: geometry collision box size=0.03 0.03 0.2; visual box size=0.03 0.03 0.2
- link back_rocker_link: geometry collision box size=0.03 0.632 0.03; visual box size=0.03 0.632 0.03
- link back_rocker_right_link: geometry collision box size=0.03 0.03 0.2; visual box size=0.03 0.03 0.2
- link backward_left_front_rocker_link: geometry collision box size=0.3 0.03 0.03; visual box size=0.3 0.03 0.03
- link backward_right_front_rocker_link: geometry collision box size=0.3 0.03 0.03; visual box size=0.3 0.03 0.03
- link base_link: geometry collision box size=0.78 0.504 0.278; visual box size=0.78 0.504 0.278
- link forward_left_front_rocker_link: geometry collision box size=0.33 0.03 0.03; visual box size=0.33 0.03 0.03
- link forward_right_front_rocker_link: geometry collision box size=0.33 0.03 0.03; visual box size=0.33 0.03 0.03
- link left_back_wheel_link: geometry collision cylinder length=0.055 radius=0.127; visual cylinder length=0.055 radius=0.127
- link left_front_wheel_link: geometry collision cylinder length=0.055 radius=0.127; visual cylinder length=0.055 radius=0.127
- link left_pneumatic_wheel_link: geometry collision cylinder length=0.055 radius=0.127; visual cylinder length=0.055 radius=0.127
- link lidar_link: geometry collision cylinder length=0.05 radius=0.1; visual cylinder length=0.05 radius=0.1
- link right_back_wheel_link: geometry collision cylinder length=0.055 radius=0.127; visual cylinder length=0.055 radius=0.127
- link right_front_wheel_link: geometry collision cylinder length=0.055 radius=0.127; visual cylinder length=0.055 radius=0.127
- link right_pneumatic_wheel_link: geometry collision cylinder length=0.055 radius=0.127; visual cylinder length=0.055 radius=0.127
- link upper_base_link: geometry collision box size=0.4 0.504 0.382; visual box size=0.4 0.504 0.382

Commit message: Added inertial tags to URDF for making compatible with Gazebo

File: src/robot_simulation/urdf/rover.urdf (robot description, URDF)
Before this commit: robot my_robot, 16 links, 15 joints
Links:
- link back_rocker_left_link: mass None -> 1.0
- link back_rocker_link: mass None -> 1.0
- link back_rocker_right_link: mass None -> 1.0
- link backward_left_front_rocker_link: mass None -> 1.0
- link backward_right_front_rocker_link: mass None -> 1.0
- link base_link: mass None -> 10.0
- link forward_left_front_rocker_link: mass None -> 1.0
- link forward_right_front_rocker_link: mass None -> 1.0
- link left_back_wheel_link: mass None -> 1.0
- link left_front_wheel_link: mass None -> 1.0
- link left_pneumatic_wheel_link: mass None -> 1.0
- link lidar_link: mass None -> 0.5
- link right_back_wheel_link: mass None -> 1.0
- link right_front_wheel_link: mass None -> 1.0
- link right_pneumatic_wheel_link: mass None -> 1.0
- link upper_base_link: mass None -> 10.0

File: src/robot_simulation/urdf/simple_robot.urdf (robot description, URDF)
Before this commit: robot simple_robot, 1 links, 0 joints
Links:
- link base_link: mass None -> 1.0; geometry collision box size=0.5 0.5 0.5; visual box size=0.5 0.5 0.5

Commit message: Added RpLidar plugin to urdf for gazebo

File: src/robot_simulation/urdf/rover.urdf (robot description, URDF)
Before this commit: robot my_robot, 16 links, 15 joints
Links:
- removed link lidar_link
- added link rplidar_link, mass 0.1; collision cylinder length=0.041 radius=0.038; visual cylinder length=0.041 radius=0.038
Joints:
- removed joint base_lidar_joint
- added joint base_rplidar_joint: type fixed, parent base_link, child rplidar_link, origin xyz=0.29 0.0 0.303 rpy=0.0 0.0 0.0
- joint base_back_rocker_joint: origin xyz=-0.425 0.0 0.0 rpy=0.0 0.0 0.0 -> xyz=-0.425 0.0 -0.028 rpy=0.0 0.0 0.0

Commit message: Added IMU sensor and plugin in URDF

File: src/robot_simulation/urdf/rover.urdf (robot description, URDF)
Before this commit: robot my_robot, 16 links, 15 joints
Links:
- added link imu_link, mass 0.1; collision box size=0.015 0.02 0.001; visual box size=0.015 0.02 0.001
Joints:
- added joint base_imu_joint: type fixed, parent base_link, child imu_link, origin xyz=0.0 0.0 0.66 rpy=0.0 0.0 0.0
