Commit message: fixed error in 4wheel drive URDF

File: src/robot_simulation/urdf/4wheel.urdf (robot description, URDF)
Before this commit: robot my_robot, 9 links, 8 joints
Joints:
- removed joint base_front_wheel_joint
- added joint base_right_front_wheel_joint: type continuous, parent base_link, child right_front_wheel_link, origin xyz=0.195 -0.3645 0.0 rpy=1.57 0.0 0.0, axis 0.0 0.0 -1.0
